Commit message: 增加了base2scan的tf转换，更完备.suc!

File: pf_localization/urdf/R2D2_base.xacro (robot description, xacro)
@@ -14,4 +14,6 @@
 <!-- the vertical offset dist bet the laser and car body -->
 <xacro:property name="up_laser" value="0.1" />
+<!-- the horizontal offset in x dir dist bet the laser and car center -->
+<xacro:property name="x_offset_laser" value="0.4" />
 <!-- the vertical offset dist bet the driving wheel and car body -->
 <xacro:property name="down_wheel" value="0.35" />
@@ -36,6 +38,6 @@
     </inertial>
   </xacro:macro>
-<!--link name="base_footprint">
-</link-->
+<link name="base_footprint">
+</link>
 <link name="base_link">
     <visual>
@@ -120,10 +122,10 @@
   <!-- published int launch file -->
   <!-- if published in here the tf time will too fast than other link ,it will display error in rviz-->
-  <!--joint name="base_footprint_to_base_link" type="fixed">
+  <joint name="base_footprint_to_base_link" type="fixed">
     <parent link="base_footprint"/>
     <child link="base_link"/>
     <origin xyz="0 0 0.5" rpy="0 0 0"/>
     <axis xyz="0 1 0"/>
-  </joint-->
+  </joint>
   <joint name="left_front_wheel_joint" type="continuous">
     <parent link="base_link"/>
@@ -152,5 +154,5 @@
   <xacro:include filename="$(find pf_localization)/urdf/hokuyolaser_base.xacro" />
   <xacro:hokuyolaser parent_link="base_link">
-    <origin xyz="0 0 ${up_z+up_laser}" rpy="0 0 0" />
+    <origin xyz="${x_offset_laser} 0 ${up_z+up_laser}" rpy="0 0 0" />
   </xacro:hokuyolaser>
 <transmission name="left_front_wheel_trans">

Commit message: 实测了建图定位程序;rfs slam err < 10mm. 并修改了程序bug(定位);SUC!

File: pf_localization/urdf/R2D2_base.xacro (robot description, xacro)
@@ -16,4 +16,8 @@
 <!-- the horizontal offset in x dir dist bet the laser and car center -->
 <xacro:property name="x_offset_laser" value="0.4" />
+<!-- the horizontal offset in y dir dist bet the laser and car center -->
+<xacro:property name="y_offset_laser" value="-0.2" />
+<!-- laser rotate angle in yaw -->
+<xacro:property name="yaw_laser" value="-1.57" />
 <!-- the vertical offset dist bet the driving wheel and car body -->
 <xacro:property name="down_wheel" value="0.35" />
@@ -154,5 +158,5 @@
   <xacro:include filename="$(find pf_localization)/urdf/hokuyolaser_base.xacro" />
   <xacro:hokuyolaser parent_link="base_link">
-    <origin xyz="${x_offset_laser} 0 ${up_z+up_laser}" rpy="0 0 0" />
+    <origin xyz="${x_offset_laser} ${y_offset_laser} ${up_z+up_laser}" rpy="0 0 ${yaw_laser}" />
   </xacro:hokuyolaser>
 <transmission name="left_front_wheel_trans">

File: pf_mapping/urdf/R2D2_base.xacro (robot description, xacro)
@@ -17,4 +17,8 @@
 <xacro:property name="x_offset_laser" value="0.4" />
 <!-- the vertical offset dist bet the driving wheel and car body -->
+<!-- the horizontal offset in y dir dist bet the laser and car center -->
+<xacro:property name="y_offset_laser" value="-0.2" />
+<!-- laser rotate angle in yaw -->
+<xacro:property name="yaw_laser" value="-1.57" />
 <xacro:property name="down_wheel" value="0.35" />
 <!-- the horizontal offset dist bet the driven wheel and car body -->
@@ -154,5 +158,5 @@
   <xacro:include filename="$(find pf_localization)/urdf/hokuyolaser_base.xacro" />
   <xacro:hokuyolaser parent_link="base_link">
-    <origin xyz="${x_offset_laser} 0 ${up_z+up_laser}" rpy="0 0 0" />
+    <origin xyz="${x_offset_laser} ${y_offset_laser} ${up_z+up_laser}" rpy="0 0 ${yaw_laser}" />
   </xacro:hokuyolaser>
 <transmission name="left_front_wheel_trans">
