Commit message: mod!

File: robotnik_purepursuit_planner-master/robotnik_pp_planner/urdf/R2D2_base.xacro (robot description, xacro)
@@ -30,4 +30,5 @@
 <xacro:property name="car_body_width" value="0.8" />
 <xacro:property name="car_body_height" value="0.1" />
+  <xacro:property name="imu_stdev" value="0.00017" />
   <xacro:macro name="default_inertial" params="mass">
     <inertial>
@@ -150,8 +151,14 @@
     <axis xyz="0 1 0"/>
   </joint>
-  <xacro:include filename="$(find robotnik_pp_planner)/urdf/hokuyolaser_base_test.xacro" />
+  <!--                   !!!scan!!!                                   -->
+  <xacro:include filename="$(find robotnik_pp_planner)/urdf/hokuyolaser_base.xacro" />
   <xacro:hokuyolaser parent_link="base_link">
     <origin xyz="0 0 ${up_z+up_laser}" rpy="0 0 0" />
   </xacro:hokuyolaser>
+ <!--                     !!!imu!!!                                  -->
+  <xacro:include filename="$(find robotnik_pp_planner)/urdf/imu.gazebo.urdf.xacro" />
+  <xacro:imu_gazebo parent_link="base_link" link="imu_link" imu_topic="imu_data" update_rate="50.0" stdev="${imu_stdev}" >
+    <origin xyz="0 0 0" rpy="0 0 0" />
+  </xacro:imu_gazebo>
 <transmission name="left_front_wheel_trans">
   <type>transmission_interface/SimpleTransmission</type>
@@ -215,4 +222,28 @@
   </plugin>
 </gazebo-->
+<!--xacro:macro name="diff_controller_plugin_gazebo" params="prefix left_wheel_joint right_wheel_joint wheel_separation wheel_radius">
+  <gazebo>
+    <plugin name="diff_drive_controller" filename="libgazebo_ros_diff_drive.so">
+      <legacyMode>false</legacyMode>
+      <alwaysOn>true</alwaysOn>
+      <updateRate>1000.0</updateRate>
+      <leftJoint>${left_wheel_joint}</leftJoint>
+      <rightJoint>${right_wheel_joint}</rightJoint>
+      <wheelSeparation>${wheel_separation}</wheelSeparation>
+      <wheelDiameter>${2*wheel_radius}</wheelDiameter>
+      <wheelTorque>10</wheelTorque>
+      <publishTf>1</publishTf>
+      <odometryFrame>map</odometryFrame>
+      <commandTopic>mobile_base_controller/cmd_vel</commandTopic>
+      <odometryTopic>mobile_base_controller/odom</odometryTopic>
+      <robotBaseFrame>base_footprint</robotBaseFrame>
+      <wheelAcceleration>2.8</wheelAcceleration>
+      <publishWheelJointState>true</publishWheelJointState>
+      <publishWheelTF>false</publishWheelTF>
+      <odometrySource>world</odometrySource>
+      <rosDebugLevel>Debug</rosDebugLevel>
+    </plugin>
+  </gazebo>
+</xacro:macro-->
  <gazebo>
   <plugin name="gazebo_ros_control" filename="libgazebo_ros_control.so">

File: robotnik_purepursuit_planner-master/robotnik_pp_planner/urdf/hokuyolaser_base.xacro (robot description, xacro)
@@ -45,5 +45,5 @@
           <range>
             <min>0.001</min>
-            <max>20.0</max>
+            <max>50.0</max>
             <resolution>0.001</resolution>resewt
           </range>
