Commit message: some mod

File: imu_odom_combine/urdf/R2D2_base.xacro (robot description, xacro)
@@ -38,6 +38,6 @@
     </inertial>
   </xacro:macro>
-<!--link name="base_footprint">
-</link-->
+<link name="base_footprint">
+</link>
 <link name="base_link">
     <visual>
@@ -122,10 +122,10 @@
   <!-- published int launch file -->
   <!-- if published in here the tf time will too fast than other link ,it will display error in rviz-->
-  <!--joint name="base_footprint_to_base_link" type="fixed">
+  <joint name="base_footprint_to_base_link" type="fixed">
     <parent link="base_footprint"/>
     <child link="base_link"/>
     <origin xyz="0 0 0.5" rpy="0 0 0"/>
     <axis xyz="0 1 0"/>
-  </joint-->
+  </joint>
   <joint name="left_front_wheel_joint" type="continuous">
     <parent link="base_link"/>

File: imu_odom_combine/urdf/R2D2_base_kf.xacro (robot description, xacro)
@@ -31,4 +31,5 @@
 <xacro:property name="car_body_width" value="0.8" />
 <xacro:property name="car_body_height" value="0.1" />
+  <!--  1deg = 0.017rad -->
   <xacro:property name="imu_stdev" value="0.00017" />
   <xacro:macro name="default_inertial" params="mass">
@@ -38,6 +39,6 @@
     </inertial>
   </xacro:macro>
-<!--link name="base_footprint">
-</link-->
+<link name="base_footprint">
+</link>
 <link name="base_link">
     <visual>
@@ -122,10 +123,10 @@
   <!-- published int launch file -->
   <!-- if published in here the tf time will too fast than other link ,it will display error in rviz-->
-  <!--joint name="base_footprint_to_base_link" type="fixed">
+  <joint name="base_footprint_to_base_link" type="fixed">
     <parent link="base_footprint"/>
     <child link="base_link"/>
     <origin xyz="0 0 0.5" rpy="0 0 0"/>
     <axis xyz="0 1 0"/>
-  </joint-->
+  </joint>
   <joint name="left_front_wheel_joint" type="continuous">
     <parent link="base_link"/>

File: imu_odom_combine/urdf/hokuyolaser_base.xacro (robot description, xacro)
@@ -46,5 +46,5 @@
             <min>0.001</min>
             <max>50.0</max>
-            <resolution>0.001</resolution>resewt
+            <resolution>0.001</resolution>
           </range>
           <noise>
