Commit message: 简化了d8_1000urdf模型.suc.增加了d8_1000的部分launch文件

File: dhc_houdar_pkg/urdf/R2D2_base.xacro (robot description, xacro)
@@ -1,4 +1,4 @@
 <?xml version="1.0"?>
-<robot name="R2D2" xmlns:xacro="http://ros.org/wiki/xacro">
+<robot name="R2D2" xmlns:xacro="http://www.ros.org/wiki/xacro">
 <material name="blue">
   <color rgba="0 0 0.8 1"/>

File: dhc_houdar_pkg/urdf/scrubot/d8_1000/caster_wheel.xacro (robot description, xacro)
@@ -1,9 +1,9 @@
 <?xml version="1.0" ?>
-<robot xmlns:xacro="http://ros.org/wiki/xacro">
+<robot xmlns:xacro="http://www.ros.org/wiki/xacro">
 <!--
   caster wheel and joints defined
 -->
-  <xacro:property name="M_PI" default="3.14159"/>
-<xacro:property name="caster_wheel_mass" value="1.0" />
+  <!--xacro:property name="M_PI" default="3.14159"/-->
+<xacro:property name="caster_wheel_mass" value="200" />
 <xacro:property name="caster_wheel_radius" value="0.05" />
 <xacro:property name="caster_wheel_width" value="0.037" />

File: dhc_houdar_pkg/urdf/scrubot/d8_1000/chassis.xacro (robot description, xacro)
@@ -1,5 +1,5 @@
 <?xml version="1.0"?>
 <robot xmlns:xacro="http://www.ros.org/wiki/xacro">
- <xacro:property name="M_PI" default="3.14159"/>
+ <!--xacro:property name="M_PI" value="3.14159"/-->
   <!-- Base Properties -->
   <xacro:property name="mass_base" value="100.0" />
@@ -9,9 +9,17 @@
   <xacro:property name="driving_wheel2base_rear_dist" value="0.075" />
   <xacro:property name="driving_wheel2ground_dist" value="0.188" />
+  <xacro:property name="crash_resistant_edge_length" value="0.76625" />
+  <xacro:property name="crash_resistant_edge_down2ground" value="0.0554" />
 <xacro:property name="base_down2ground" value="0.156" />
-  <!-- the vertical offset dist bet the car and the ground -->
+  <!--
+  the vertical offset dist bet the car and the ground
   <xacro:property name="offset_x" value="-0.32362" />
   <xacro:property name="offset_y" value="-0.443" />
   <xacro:property name="offset_z" value="-0.045" />
+  -->
+  <!-- conf for chassis_simple.stl -->
+<xacro:property name="offset_x" value="${-driving_wheel2base_rear_dist}" />
+<xacro:property name="offset_y" value="${-crash_resistant_edge_length/2}" />
+<xacro:property name="offset_z" value="${crash_resistant_edge_down2ground}" />
  <xacro:macro name="default_inertial" params="mass">
     <inertial>
@@ -29,7 +37,5 @@
           <!--box size="${base_x_size} ${base_y_size} ${base_z_size}" /-->
         </geometry>
-        <material name="grey">
-          <color rgba="0.6 0.6 0.6 1"/>
-        </material>
+        <xacro:insert_block name="material_Azure2" />
       </visual>
       <collision>
@@ -50,5 +56,5 @@
     </joint>
     <gazebo reference="${name}">
-      <material>Gazebo/Grey</material>
+      <material>Gazebo/Blue</material>
     </gazebo>
   </xacro:macro>

File: dhc_houdar_pkg/urdf/scrubot/d8_1000/d8_1000.xacro (robot description, xacro)
@@ -1,4 +1,5 @@
 <?xml version="1.0"?>
-<robot name="d8_1000" xmlns:xacro="http://ros.org/wiki/xacro">
+<robot name="d8_1000" xmlns:xacro="http://www.ros.org/wiki/xacro">
+<xacro:property name="M_PI" value="3.1415926"/>
 <xacro:property name="pkg" value="$(find dhc_houdar_pkg)/urdf/scrubot/d8_1000" />
 <xacro:property name="mesh_dir" value="package://dhc_houdar_pkg/urdf/scrubot/d8_1000/mesh"/>
@@ -18,10 +19,10 @@
 <xacro:property name="base_link_name" value="base_link"/>
 <!-- body -->
-<xacro:chassis  name="${base_link_name}" parent_link="${base_name}" meshes="${mesh_dir}/chassis.stl"  >
+<xacro:chassis  name="${base_link_name}" parent_link="${base_name}" meshes="${mesh_dir}/chassis_simple.stl"  >
 </xacro:chassis>
 <!-- driving wheel -->
-<xacro:driving_wheel wheel_prefix="left" parent_link="${base_link_name}" left_right="1" mesh="${mesh_dir}/driving_wheel.stl" >
+<xacro:driving_wheel wheel_prefix="left" parent_link="${base_link_name}" left_right="1" mesh="${mesh_dir}/driving_wheel_surface.stl" >
  </xacro:driving_wheel>
-<xacro:driving_wheel wheel_prefix="right" parent_link="${base_link_name}" left_right="-1" mesh="${mesh_dir}/driving_wheel.stl" >
+<xacro:driving_wheel wheel_prefix="right" parent_link="${base_link_name}" left_right="-1" mesh="${mesh_dir}/driving_wheel_surface.stl" >
  </xacro:driving_wheel>
 <!-- caster wheel -->

File: dhc_houdar_pkg/urdf/scrubot/d8_1000/driving_wheel.xacro (robot description, xacro)
@@ -1,5 +1,5 @@
 <?xml version="1.0"?>
 <robot xmlns:xacro="http://www.ros.org/wiki/xacro">
-  <xacro:property name="M_PI" default="3.14159"/>
+  <!--xacro:property name="M_PI" value="3.14159"/-->
   <!-- Wheel Properties -->
   <xacro:property name="wheel_separation" value="0.64" />
@@ -29,5 +29,5 @@
          <!-- cylinder length="${driving_wheel_width}" radius="${driving_wheel_radius}"/ -->
         </geometry>
-        <xacro:insert_block name="material_dark_grey" />
+        <xacro:insert_block name="material_yellow" />
       </visual>
       <collision>

File: dhc_houdar_pkg/urdf/scrubot/d8_1000/gazebo.xacro (robot description, xacro)
@@ -1,4 +1,4 @@
 <?xml version="1.0" ?>
-<robot xmlns:xacro="http://ros.org/wiki/xacro">
+<robot xmlns:xacro="http://www.ros.org/wiki/xacro">
   <gazebo>
    <plugin name="gazebo_ros_control" filename="libgazebo_ros_control.so">

File: dhc_houdar_pkg/urdf/scrubot/d8_1000/inertial.xacro (robot description, xacro)
@@ -3,6 +3,6 @@
   see https://github.com/uos/uos_tools/blob/fuerte/uos_common_urdf/common.xacro and
   see http://answers.gazebosim.org/question/4372/the-inertia-matrix-explained/ -->
-<robot xmlns:xacro="http://ros.org/wiki/xacro">
-  <property name="M_PI" value="3.1415926535897931" />
+<robot xmlns:xacro="http://www.ros.org/wiki/xacro">
+  <!--xacro:property name="M_PI" value="3.1415926535897931" /-->
   <!-- see https://secure.wikimedia.org/wikipedia/en/wiki/List_of_moment_of_inertia_tensors -->
   <!-- #################### versions without origin #################### -->

File: dhc_houdar_pkg/urdf/scrubot/d8_1000/materials.xacro (robot description, xacro)
@@ -3,5 +3,5 @@
   Various useful properties such as constants and materials
  -->
-<robot name="d8_1000_properties" xmlns:xacro="http://ros.org/wiki/xacro">
+<robot name="d8_1000_properties" xmlns:xacro="http://www.ros.org/wiki/xacro">
   <!-- #################### RViz materials #################### -->
   <xacro:property name="material_white">
@@ -12,5 +12,5 @@
   <xacro:property name="material_yellow">
     <material name="yellow">
-      <color rgba="${255/255} ${226/255} ${0/255} 1"/>
+      <color rgba="1 0.886 0 1"/>
     </material>
   </xacro:property>
@@ -55,3 +55,13 @@
     </material>
   </xacro:property>
+<xacro:property name="material_blue">
+  <material name="ChassisBlue">
+    <color rgba="0 0 1 0.5" />
+  </material>
+</xacro:property>
+<xacro:property name="material_Azure2">
+  <material name="ChassisAzure2">
+    <color rgba="0.003921 0.933 0.933 0.7" />
+  </material>
+</xacro:property>
 </robot>

File: dhc_houdar_pkg/urdf/scrubot/d8_1000/sensor/imu.xacro (robot description, xacro)
@@ -1,4 +1,4 @@
 <?xml version="1.0"?>
-<robot xmlns:xacro="http://ros.org/wiki/xacro">
+<robot xmlns:xacro="http://www.ros.org/wiki/xacro">
 <xacro:macro name="imu_gazebo" params="parent_link link imu_topic update_rate stdev *joint_origin">
 <!-- 1,create link -->

File: dhc_houdar_pkg/urdf/scrubot/d8_1000/sensor/sick_551.xacro (robot description, xacro)
@@ -2,5 +2,4 @@
 <robot xmlns:xacro="http://www.ros.org/wiki/xacro">
 <!-- chq define the laser glass cylinbe center is the laser cord center -->
- <xacro:property name="M_PI" default="3.14159"/>
  <xacro:property name="laser_rect_x" value="0.059" />
   <xacro:property name="laser_glass_radius" value="0.051" />
@@ -26,7 +25,8 @@
           <mesh filename="${mesh}"/>
         </geometry>
+        <xacro:insert_block name="material_light_grey" />
       </visual>
       <inertial>
-        <mass value="2" />
+        <mass value="0.1" />
        <origin xyz="${-laser_rect_x} ${-laser_glass_radius} ${laser_glass_thick/2.0-laser_z}" rpy="0 0 0"/>
         <inertia ixx="1e-6" ixy="0" ixz="0" iyy="1e-6" iyz="0" izz="1e-6" />
@@ -35,5 +35,5 @@
   <!-- laser -->
     <gazebo reference="${name}_link">
-      <material>Gazebo/Black</material>
+      <material>Gazebo/Grey</material>
       <sensor type="gpu_ray" name="head_laser_sensor">
     <!--sensor type="ray" name="head_hokuyo_sensor"-->
@@ -47,6 +47,6 @@
               <samples>720</samples>
               <resolution>0.5</resolution>
-              <min_angle>-1.5707963</min_angle>
-              <max_angle>1.5707963</max_angle>
+              <min_angle>${-M_PI/2}</min_angle>
+              <max_angle>${M_PI/2}</max_angle>
             </horizontal>
           </scan>

File: dhc_houdar_pkg/urdf/scrubot/d8_1000/sensor/sonar_ks106.xacro (robot description, xacro)
@@ -1,4 +1,4 @@
 <?xml version="1.0"?>
-<robot xmlns:xacro="http://ros.org/wiki/xacro">
+<robot xmlns:xacro="http://www.ros.org/wiki/xacro">
   <xacro:property name="sonar_base_x" value="0.361" />
   <xacro:property name="sonar_base_y" value="0.0" />
