Commit message: 修改了配重，确保从车子在未发送指令的情况下静止.suc!

File: dhc_houdar_pkg/urdf/scrubot/d8_1000/caster_wheel.xacro (robot description, xacro)
@@ -5,5 +5,5 @@
 -->
   <!--xacro:property name="M_PI" default="3.14159"/-->
-<xacro:property name="caster_wheel_mass" value="200" />
+<xacro:property name="caster_wheel_mass" value="1" />
 <xacro:property name="caster_wheel_radius" value="0.05" />
 <xacro:property name="caster_wheel_width" value="0.037" />
@@ -78,5 +78,5 @@
     <child link="${wheel_prefix}_caster_rotation_link" />
     <axis xyz="0 0 1" />
-    <dynamics damping="0.01" friction="0.0"/>
+    <dynamics damping="0.05" friction="0.1"/>
   </joint>
  <!-- caster wheel to catster rotation joint-->

File: dhc_houdar_pkg/urdf/scrubot/d8_1000/chassis.xacro (robot description, xacro)
@@ -3,5 +3,5 @@
  <!--xacro:property name="M_PI" value="3.14159"/-->
   <!-- Base Properties -->
-  <xacro:property name="mass_base" value="100.0" />
+  <xacro:property name="mass_base" value="200.0" />
   <xacro:property name="base_x_size" value="0.6" />
   <xacro:property name="base_y_size" value="0.57" />

File: dhc_houdar_pkg/urdf/scrubot/d8_1000/driving_wheel.xacro (robot description, xacro)
@@ -7,5 +7,5 @@
   <xacro:property name="driving_wheel_width" value="0.065" />
   <xacro:property name="driving_wheel_radius" value="${wheel_radius}" />
-  <xacro:property name="mass_driving_wheel" value="0.5" />
+  <xacro:property name="mass_driving_wheel" value="3" />
   <xacro:property name="mechanicalReductionRatio" value ="21.0" />
   <xacro:property name="driving_wheel_base_dx" value="0.0" />
@@ -44,5 +44,5 @@
     </gazebo>
     <!-- gazebo dynamics-->
-    <!--gazebo reference="${wheel_prefix}_driving_wheel_link">
+    <gazebo reference="${wheel_prefix}_driving_wheel_link">
       <mu1 value="1.0"/>
       <mu2 value="1.0"/>
@@ -50,5 +50,5 @@
       <kd value="1.0" />
       <fdir1 value="1 0 0"/>
-  </gazebo-->
+  </gazebo>
      <!-- joint -->
     <joint name="${wheel_prefix}_driving_wheel_joint" type="continuous">
